Commit message: Tweeks

File: notebooks/ros_urdf/.ipynb_checkpoints/model.urdf-checkpoint.xacro (robot description, xacro)
@@ -1,8 +1,4 @@
 <?xml version="1.0"?>
-<robot name="efim"
-       xmlns:sensor="http://playerstage.sourceforge.net/gazebo/xmlschema/#sensor"
-       xmlns:controller="http://playerstage.sourceforge.net/gazebo/xmlschema/#controller"
-       xmlns:interface="http://playerstage.sourceforge.net/gazebo/xmlschema/#interface"
-       xmlns:xacro="http://ros.org/wiki/xacro">
+<robot name="efim" xmlns:sensor="http://playerstage.sourceforge.net/gazebo/xmlschema/#sensor" xmlns:controller="http://playerstage.sourceforge.net/gazebo/xmlschema/#controller" xmlns:interface="http://playerstage.sourceforge.net/gazebo/xmlschema/#interface" xmlns:xacro="http://ros.org/wiki/xacro">
   <!-- BASE-FOOTPRINT -->
   <!-- base_footprint is a fictitious link(frame) that is on the ground right below base_link origin -->
@@ -11,18 +7,16 @@
       <mass value="0.0001" />
       <origin xyz="0 0 0" />
-      <inertia ixx="0.0001" ixy="0.0" ixz="0.0"
-          iyy="0.0001" iyz="0.0"
-          izz="0.0001" />
-    </inertial>
-    <visual>
-        <origin xyz="0 0 0" rpy="0 0 0" />
-        <geometry>
-            <box size="0.001 0.001 0.001" />
-        </geometry>
+      <inertia ixx="0.0001" ixy="0.0" ixz="0.0" iyy="0.0001" iyz="0.0" izz="0.0001" />
+    </inertial>
+    <visual>
+      <origin xyz="0 0 0" rpy="0 0 0" />
+      <geometry>
+        <box size="0.001 0.001 0.001" />
+      </geometry>
     </visual>
   </link>
   <joint name="base_footprint_joint" type="fixed">
-    <origin xyz="0 0 0" rpy="0 0 0" />
-    <parent link="base_footprint"/>
+    <origin xyz="0 0 0.0762" rpy="0 0 0" />
+    <parent link="base_footprint" />
     <child link="base_link" />
   </joint>
@@ -30,19 +24,18 @@
     <visual>
       <geometry>
-        <box size="0.41148 0.30988 0.05588"/>
+        <box size="0.41148 0.30988 0.05588" />
       </geometry>
       <material name="grey">
-	<color rgba="0.5 0.5 0.5 1"/>
-      </material>
-    </visual>
-    <collision>
-      <geometry>
-        <box size="0.41148 0.30988 0.05588"/>
-      </geometry>
-    </collision>
-   <inertial>
-      <mass value="20.0"/>
-      <inertia ixx="1.0" iyy="1.0" izz="1.0"
-               ixy="0" ixz="0" iyz="0"/>
+        <color rgba="0.5 0.5 0.5 1" />
+      </material>
+    </visual>
+    <collision>
+      <geometry>
+        <box size="0.41148 0.30988 0.05588" />
+      </geometry>
+    </collision>
+    <inertial>
+      <mass value="20.0" />
+      <inertia ixx="1.0" iyy="1.0" izz="1.0" ixy="0" ixz="0" iyz="0" />
     </inertial>
   </link>
@@ -53,76 +46,74 @@
     <visual>
       <geometry>
+        <cylinder length="1.04775" radius="0.2032" />
+      </geometry>
+      <material name="clear">
+        <color rgba="0.75 0.75 0.75 0.4" />
+      </material>
+    </visual>
+    <!--<collision>
+      <geometry>
         <cylinder length="1.04775" radius="0.2032"/>
       </geometry>
-      <material name="clear">
-        <color rgba="0.75 0.75 0.75 0.4"/>
+    </collision>-->
+    <inertial>
+      <mass value="10.0" />
+      <inertia ixx="1.0" iyy="1.0" izz="1.0" ixy="0" ixz="0" iyz="0" />
+    </inertial>
+  </link>
+  <joint name="center_joint" type="fixed">
+    <axis xyz="0 0 1" />
+    <parent link="base_link" />
+    <child link="body_link" />
+    <origin rpy="0 0 0" xyz="0 0 0.551815" />
+  </joint>
+  <link name="camera_link">
+    <visual>
+      <origin rpy="0 0 0" />
+      <geometry>
+        <box size="0.0762 0.2794 0.0762" />
+      </geometry>
+      <material name="red">
+        <color rgba="1 0.1 0.1 1" />
       </material>
     </visual>
     <!--<collision>
       <geometry>
-        <cylinder length="1.04775" radius="0.2032"/>
+        <box size="0.0762 0.2794 0.0762"/>
       </geometry>
     </collision>-->
     <inertial>
-      <mass value="10.0"/>
-      <inertia ixx="1.0" iyy="1.0" izz="1.0"
-               ixy="0" ixz="0" iyz="0"/>
-    </inertial>
-  </link>
-  <joint name="center_joint" type="fixed">
-    <axis xyz="0 0 1"/>
-    <parent link="base_link"/>
-    <child link="body_link"/>
-    <origin rpy="0 0 0" xyz="0 0 0.551815"/>
-  </joint>
-  <link name="camera_link">
-    <visual>
-      <origin rpy="0 0 0"/>
-      <geometry>
-        <box size="0.0762 0.2794 0.0762"/>
-      </geometry>
-      <material name="red">
-	<color rgba="1 0.1 0.1 1"/>
-      </material>
-    </visual>
-    <!--<collision>
-      <geometry>
-        <box size="0.0762 0.2794 0.0762"/>
-      </geometry>
-    </collision>-->
-   <inertial>
-      <mass value="0.25"/>
-      <inertia ixx="1.0" iyy="1.0" izz="1.0"
-               ixy="0" ixz="0" iyz="0"/>
+      <mass value="0.25" />
+      <inertia ixx="1.0" iyy="1.0" izz="1.0" ixy="0" ixz="0" iyz="0" />
     </inertial>
   </link>
   <joint name="camera_joint" type="fixed">
-    <axis xyz="0 0 0"/>
-    <parent link="base_link"/>
-    <child link="camera_link"/>
-    <origin rpy="0 0 0" xyz="0.15 0 0.48"/>
-  </joint>
-    <!-- The fixed joints & links below are usually published by static_transformers launched by the OpenNi launch
+    <axis xyz="0 1 0" />
+    <parent link="base_link" />
+    <child link="camera_link" />
+    <origin rpy="0 0 0" xyz="0.15 0 0.48" />
+  </joint>
+  <!-- The fixed joints & links below are usually published by static_transformers launched by the OpenNi launch
          files. However, for Gazebo simulation we need them, so we add them here.
          (Hence, don't publish them additionally!) -->
-	<joint name="camera_depth_joint" type="fixed">
-	  <origin xyz="0 0 0" rpy="0 0 0" />
-	  <parent link="camera_link" />
-	  <child link="camera_depth_frame" />
-	</joint>
-	<link name="camera_depth_frame"/>
-	<joint name="camera_depth_optical_joint" type="fixed">
-	  <origin xyz="0 0 0" rpy="0 0 0" />
-	  <parent link="camera_link" />
-	  <child link="camera_depth_optical_frame" />
-	</joint>
-	<link name="camera_depth_optical_frame"/>
+  <joint name="camera_depth_joint" type="fixed">
+    <origin xyz="0 1 0" rpy="-1.5708 0 -1.5708" />
+    <parent link="camera_link" />
+    <child link="camera_depth_frame" />
+  </joint>
+  <link name="camera_depth_frame" />
+  <joint name="camera_depth_optical_joint" type="fixed">
+    <origin xyz="0 0 0" rpy="0 0 0" />
+    <parent link="camera_link" />
+    <child link="camera_depth_optical_frame" />
+  </joint>
+  <link name="camera_depth_optical_frame" />
   <link name="laser">
     <visual>
       <geometry>
-        <box size="0.0762 0.0762 0.0762"/>
+        <box size="0.0762 0.0762 0.0762" />
       </geometry>
       <material name="blue">
-	<color rgba="0.1 0.1 1 1"/>
+        <color rgba="0.1 0.1 1 1" />
       </material>
     </visual>
@@ -132,150 +123,149 @@
       </geometry>
     </collision>-->
-   <inertial>
-      <mass value="0.25"/>
-      <inertia ixx="1.0" iyy="1.0" izz="1.0"
-               ixy="0" ixz="0" iyz="0"/>
+    <inertial>
+      <mass value="0.25" />
+      <inertia ixx="1.0" iyy="1.0" izz="1.0" ixy="0" ixz="0" iyz="0" />
     </inertial>
   </link>
   <joint name="laser_joint" type="fixed">
-    <axis xyz="0 0 1"/>
-    <parent link="base_link"/>
-    <child link="laser"/>
-    <origin rpy="0 0 0" xyz="0.0 0 1.23"/>
-  </joint>
-  <link name="front_sonar">
-    <visual>
-      <geometry>
-        <box size="0.04 0.04 0.04"/>
-      </geometry>
-      <material name="red">
-   <inertial>
-      <mass value="0.25"/>
-      <inertia ixx="1.0" iyy="1.0" izz="1.0"
-               ixy="0" ixz="0" iyz="0"/>
-    </inertial>
-  </link>
-  <joint name="front_sonar_link" type="continuous">
-    <axis xyz="0 0 1"/>
-    <parent link="body_link"/>
-    <child link="front_sonar"/>
-    <origin rpy="0 0 0" xyz="0.0 0.2 0.5"/>
-  </joint>
-  <link name="hitch_front_link">
-    <visual>
-      <geometry>
-        <cylinder length="0.1524" radius="0.01"/>
-      </geometry>
-      <material name="silver">
-	<color rgba="0.75 0.75 0.75 1"/>
-      </material>
-    </visual>
-    <collision>
-      <geometry>
-        <cylinder length="0.1524" radius="0.01"/>
-      </geometry>
-    </collision>
-    <inertial>
-      <mass value="0.1"/>
-      <inertia ixx="1.0" iyy="1.0" izz="1.0"
-               ixy="0" ixz="0" iyz="0"/>
-    </inertial>
-  </link>
-  <joint name="hitch_joint" type="fixed">
-    <axis xyz="0 0 1"/>
-    <parent link="base_link"/>
-    <child link="hitch_front_link"/>
-    <origin rpy="0 0 0" xyz="0.18 0 0.0762"/>
+    <axis xyz="0 0 1" />
+    <parent link="base_link" />
+    <child link="laser" />
+    <origin rpy="0 0 0" xyz="0.0 0 1.23" />
+  </joint>
+  <link name="wheel_right">
+    <visual>
+      <geometry>
+        <cylinder length="0.0508" radius="0.0762" />
+      </geometry>
+      <material name="black" />
+    </visual>
+    <collision>
+      <geometry>
+        <cylinder length="0.0508" radius="0.0762" />
+      </geometry>
+    </collision>
+    <inertial>
+      <mass value="0.1" />
+      <inertia ixx="1.0" iyy="1.0" izz="1.0" ixy="0" ixz="0" iyz="0" />
+    </inertial>
+  </link>
+  <joint name="axis_right" type="continuous">
+    <axis xyz="0 0 1" />
+    <parent link="base_link" />
+    <child link="wheel_right" />
+    <origin rpy="-1.5708 0 0" xyz="0 -0.18034 0" />
+  </joint>
+  <link name="wheel_left">
+    <visual>
+      <geometry>
+        <cylinder length="0.0508" radius="0.0762" />
+      </geometry>
+      <material name="black">
+        <color rgba="0 0 0 1" />
+      </material>
+    </visual>
+    <collision>
+      <geometry>
+        <cylinder length="0.0508" radius="0.0762" />
+      </geometry>
+    </collision>
+    <inertial>
+      <mass value="0.1" />
+      <inertia ixx="1.0" iyy="1.0" izz="1.0" ixy="0" ixz="0" iyz="0" />
+    </inertial>
+  </link>
+  <joint name="axis_left" type="continuous">
+    <axis xyz="0 0 1" />
+    <parent link="base_link" />
+    <child link="wheel_left" />
+    <origin rpy="-1.5708 0 0" xyz="0 0.18034 0" />
   </joint>
   <link name="wheel_front_left">
     <visual>
       <geometry>
-        <cylinder length="0.0508" radius="0.0762"/>
+        <cylinder length="0.0508" radius="0.0762" />
       </geometry>
       <material name="black">
-        <color rgba="0 0 0 1"/>
-      </material>
-    </visual>
-    <collision>
-      <geometry>
-        <cylinder length="0.0508" radius="0.0762"/>
-      </geometry>
-    </collision>
-    <inertial>
-      <mass value="0.1"/>
-      <inertia ixx="1.0" iyy="1.0" izz="1.0"
-               ixy="0" ixz="0" iyz="0"/>
+        <color rgba="0 0 0 1" />
+      </material>
+    </visual>
+    <collision>
+      <geometry>
+        <cylinder length="0.0508" radius="0.0762" />
+      </geometry>
+    </collision>
+    <inertial>
+      <mass value="0.1" />
+      <inertia ixx="1.0" iyy="1.0" izz="1.0" ixy="0" ixz="0" iyz="0" />
     </inertial>
   </link>
   <joint name="axis_front_left" type="continuous">
-    <axis xyz="0 0 1"/>
-    <parent link="base_link"/>
-    <child link="wheel_front_left"/>
-    <origin rpy="-1.5708 0 0" xyz="0.165862 0.18034 0"/>
-  </joint>
- <link name="wheel_front_right">
-    <visual>
-      <geometry>
-        <cylinder length="0.0508" radius="0.0762"/>
-      </geometry>
-      <material name="black"/>
-    </visual>
-    <collision>
-      <geometry>
-        <cylinder length="0.0508" radius="0.0762"/>
-      </geometry>
-    </collision>
-    <inertial>
-      <mass value="0.1"/>
-      <inertia ixx="1.0" iyy="1.0" izz="1.0"
-               ixy="0" ixz="0" iyz="0"/>
+    <axis xyz="0 0 1" />
+    <parent link="base_link" />
+    <child link="wheel_front_left" />
+    <origin rpy="-1.5708 0 0" xyz="0.165862 0.18034 0" />
+  </joint>
+  <link name="wheel_front_right">
+    <visual>
+      <geometry>
+        <cylinder length="0.0508" radius="0.0762" />
+      </geometry>
+      <material name="black" />
+    </visual>
+    <collision>
+      <geometry>
+        <cylinder length="0.0508" radius="0.0762" />
+      </geometry>
+    </collision>
+    <inertial>
+      <mass value="0.1" />
+      <inertia ixx="1.0" iyy="1.0" izz="1.0" ixy="0" ixz="0" iyz="0" />
     </inertial>
   </link>
   <joint name="axis_front_right" type="continuous">
-    <axis xyz="0 0 1"/>
-    <parent link="base_link"/>
-    <child link="wheel_front_right"/>
-    <origin rpy="-1.5708 0 0" xyz="0.165862 -0.18034 0"/>
+    <axis xyz="0 0 1" />
+    <parent link="base_link" />
+    <child link="wheel_front_right" />
+    <origin rpy="-1.5708 0 0" xyz="0.165862 -0.18034 0" />
   </joint>
   <link name="wheel_rear_right">
     <visual>
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